Commit message: Removed friction overlapping in URDF.

File: Code/Simulation/urdf/balancio_v1.urdf (robot description, URDF)
Before this commit: robot balancio, 5 links, 4 joints
Joints:
- joint joint_left_gb: limit effort=0.8 velocity=30 -> (none)
- joint joint_right_gb: limit effort=0.8 velocity=30 -> (none)
