Commit message: Changed (simplified) wheel collision shape.

File: Code/Simulation/urdf/balancio_v3.urdf (robot description, URDF)
Before this commit: robot balancio, 5 links, 4 joints
Links:
- link link_left_wheel: geometry collision cylinder length=0.25 radius=0.325; visual mesh filename=package://Code/Simulation/stl/Wheel.stl scale=10 10 10
- link link_right_wheel: geometry collision cylinder length=0.25 radius=0.325; visual mesh filename=package://Code/Simulation/stl/Wheel.stl scale=10 10 10

Commit message: Added IMU link, for real-sim compatibility.

File: Code/Simulation/urdf/balancio_v3.urdf (robot description, URDF)
Before this commit: robot balancio, 5 links, 4 joints
Links:
- added link link_IMU, mass 0.2; collision box size=0.21 0.16 0.02
Joints:
- added joint joint_IMU: type fixed, parent link_chassis, child link_IMU, origin xyz=0 0 -0.328 rpy=0 0 0
